File: kicad/ebbe34.kicad_pcb (KiCad board)
At the start: 2 copper layers, 250.3 x 111.4 mm, 93 parts, among them SW1 SW_SPDT, U2 nice_nano

Commit message: redo outline
Parts:
- removed the ? at (271.0, 59.9)
- removed the ? at (41.2, 107.2)
- removed the ? at (287.9, 107.3)
- removed the REF** at (270.9, 59.9)
- removed the REF** at (287.9, 107.3)
- removed the REF** at (198.9, 130.3)
- removed the REF** at (164.6, 158.0)
- removed the REF** at (96.3, 112.7)
- removed the REF** at (130.3, 130.3)
- removed the REF** at (41.2, 107.2)
- added ?: , , F.Cu at (263.8, 108.0)
- added ?: , , F.Cu at (159.2, 90.3)
- added ?: , , F.Cu at (170.4, 90.3)
- added ?: , , F.Cu at (91.2, 111.0)
- added ?: , , F.Cu at (65.2, 108.0)
- added REF**: Standoff_M2x6mm, ScottoKeebs_Scotto:Standoff_M2x6mm, F.Cu at (263.8, 108.0)
- added REF**: Standoff_M2x6mm, ScottoKeebs_Scotto:Standoff_M2x6mm, F.Cu at (170.4, 90.3)
- added REF**: Standoff_M2x6mm, ScottoKeebs_Scotto:Standoff_M2x6mm, F.Cu at (65.2, 108.0)
- added REF**: Standoff_M2x6mm, ScottoKeebs_Scotto:Standoff_M2x6mm, F.Cu at (91.2, 111.0)
- added REF**: Standoff_M2x6mm, ScottoKeebs_Scotto:Standoff_M2x6mm, F.Cu at (262.7, 59.5)
- added REF**: Standoff_M2x6mm, ScottoKeebs_Scotto:Standoff_M2x6mm, F.Cu at (159.2, 90.3)
- moved SW1 12.3 mm to (164.8, 85.5), turned to 180 degrees
- moved REF** 8.22 mm to (66.4, 59.5)
- moved ? 5.47 mm to (237.9, 111.0)
- moved REF** 5.47 mm to (237.9, 111.0)
- moved REF** 2.49 mm to (164.8, 90.3)
- moved REF** 1.33 mm to (127.9, 152.7)
- moved REF** 1.24 mm to (201.2, 152.7)
- moved ? 0.48 mm to (213.1, 62.6)
- moved REF** 0.48 mm to (213.1, 62.6)
- moved REF** 0.48 mm to (116.0, 62.6)
Routing:
- net RAW: track 29.0 -> 21.5 mm
- net Bat+: track 14.7 -> 9.96 mm
Other:
- board size 250.3 x 111.4 mm -> 249.3 x 112.9 mm
