File: plate/top/top.kicad_pcb (KiCad board)
At the start: 2 copper layers, 249.3 x 113.4 mm, 48 parts

Commit message: move screws
Parts:
- removed the ? at (86.6, 122.0)
- removed the ? at (209.7, 122.0)
- removed the REF** at (209.7, 122.0)
- removed the REF** at (86.6, 122.0)
- removed the REF** at (184.8, 154.1)
- removed the REF** at (111.5, 154.1)
- added ?: , , F.Cu at (158.0, 154.5)
- added ?: , , B.Cu at (158.0, 154.5)
- added REF**: Standoff_M2x6mm, ScottoKeebs_Scotto:Standoff_M2x6mm, F.Cu at (95.2, 132.7)
- added REF**: Standoff_M2x6mm, ScottoKeebs_Scotto:Standoff_M2x6mm, F.Cu at (138.3, 154.5)
- added REF**: Standoff_M2x6mm, ScottoKeebs_Scotto:Standoff_M2x6mm, F.Cu at (158.0, 154.5)
- added REF**: Standoff_M2x6mm, ScottoKeebs_Scotto:Standoff_M2x6mm, F.Cu at (201.1, 132.7)

Commit message: restore bottom curvature
Parts:
- removed the ? at (158.0, 154.5) (x2)
- removed the REF** at (138.3, 154.5)
- removed the REF** at (158.0, 154.5)
- added ?: , , F.Cu at (148.3, 159.3)
- added REF**: Standoff_M2x6mm, ScottoKeebs_Scotto:Standoff_M2x6mm, F.Cu at (148.3, 159.3)
Other:
- board size 249.3 x 113.4 mm -> 249.3 x 113.1 mm
